Commit message: Driving the Simulation robo in gazebo using teleoperation

File: description/robot.urdf.xacro (robot description, xacro)
@@ -3,3 +3,4 @@
     <!-- Example include file -->
     <xacro:include filename="robot_core.xacro" />
+    <xacro:include filename="gazebo_control.xacro"/>
 </robot>

File: description/robot_core.xacro (robot description, xacro)
@@ -41,9 +41,12 @@
         </xacro:inertial_box>
     </link>
+    <gazebo reference="chasis">
+        <material>Gazebo/White</material>
+    </gazebo>
     <!-- LEFT WHEEL -->
     <joint name="left_wheel_joint" type="continuous">
         <parent link="base_link"/>
         <child link="left_wheel"/>
-        <origin xyz="0 0.095 0" rpy="-${pi/2} 0 0"/>
+        <origin xyz="0 0.095 0" rpy="-${pi/2} 0 0" />
         <axis xyz="0 0 1"/>
     </joint>
@@ -51,5 +54,5 @@
         <visual>
             <geometry>
-                <cylinder length="0.03" radius="0.035" />
+                <cylinder length="0.03" radius="0.0335" />
             </geometry>
             <material name="blue"/>
@@ -57,11 +60,14 @@
         <collision>
             <geometry>
-                <cylinder length="0.03" radius="0.035" />
+                <cylinder length="0.03" radius="0.0335" />
             </geometry>
         </collision>
-        <xacro:inertial_cylinder mass="0.1" length="0.03" radius="0.035">
+        <xacro:inertial_cylinder mass="0.1" length="0.03" radius="0.0335">
             <origin xyz="0 0 0" rpy="0 0 0"/>
         </xacro:inertial_cylinder>
     </link>
+    <gazebo reference="left_wheel">
+        <material>Gazebo/Blue</material>
+    </gazebo>
     <!-- RIGHT WHEEL -->
     <joint name="right_wheel_joint" type="continuous">
@@ -74,5 +80,5 @@
         <visual>
             <geometry>
-                <cylinder length="0.03" radius="0.035" />
+                <cylinder length="0.03" radius="0.0335" />
             </geometry>
             <material name="blue"/>
@@ -80,11 +86,14 @@
         <collision>
             <geometry>
-                <cylinder length="0.03" radius="0.035" />
+                <cylinder length="0.03" radius="0.0335" />
             </geometry>
         </collision>
-        <xacro:inertial_cylinder mass="0.1" length="0.03" radius="0.035">
+        <xacro:inertial_cylinder mass="0.1" length="0.03" radius="0.0335">
             <origin xyz="0 0 0" rpy="0 0 0"/>
         </xacro:inertial_cylinder>
     </link>
+    <gazebo reference="right_wheel">
+        <material>Gazebo/Blue</material>
+    </gazebo>
     <!-- CASTER WHEEL -->
     <joint name="caster_wheel_joint" type="fixed">
@@ -109,3 +118,8 @@
         </xacro:inertial_sphere>
     </link>
+    <gazebo reference="caster_wheel">
+        <material>Gazebo/Black</material>
+        <mu1 value="0.001"/>
+        <mu2 value="0.001"/>
+    </gazebo>
 </robot>

Commit message: RPlidar

File: description/robot.urdf.xacro (robot description, xacro)
@@ -4,3 +4,4 @@
     <xacro:include filename="robot_core.xacro" />
     <xacro:include filename="gazebo_control.xacro"/>
+    <xacro:include filename="lidar.xacro"/>
 </robot>

File: description/robot_core.xacro (robot description, xacro)
@@ -13,4 +13,7 @@
     <material name="black">
         <color rgba="0 0 0 1"/>
+    </material>
+    <material name="red">
+        <color rgba="1 0 0 1"/>
     </material>
     <!-- base link -->
