Commit message: Robot launch file, gazedo sim, robot teleop drive

File: description/lidar.xacro (robot description, xacro)
@@ -23,6 +23,5 @@
     </link>
     <gazebo reference="laser_frame">
-        <material>Gazebo/Red</material>
-        <sensor name="laser" type="ray">
+        <sensor type="ray" name="laser">
             <pose> 0 0 0 0 0 0 </pose>
             <visualize>true</visualize>
@@ -38,5 +37,5 @@
                 <range>
                     <min>0.3</min>
-                    <max>12</max>
+                    <max>12.0</max>
                 </range>
             </ray>

File: description/ros2_control.xacro (robot description, xacro)
@@ -1,4 +1,34 @@
 <?xml version="1.0"?>
 <robot xmlns:xacro="http://www.ros.org/wiki/xacro">
+    <ros2_control name="RealRobot" type="system">
+        <hardware>
+            <plugin>diffdrive_arduino/DiffDriveArduino</plugin>
+            <param name="left_wheel_name">left_wheel_joint</param>
+            <param name="right_wheel_name">right_wheel_joint</param>
+            <param name="loop_rate">30</param>
+            <param name="device">/dev/ttyACM0</param>
+            <param name="baud_rate">57600</param>
+            <param name="timeout">1000</param>
+            <param name="enc_counts_per_rev">720</param>
+        </hardware>
+        <!-- Note everything below here is the same as the Gazebo one -->
+        <joint name="left_wheel_joint">
+            <command_interface name="velocity">
+                <param name="min">-10</param>
+                <param name="max">10</param>
+            </command_interface>
+            <state_interface name="velocity"/>
+            <state_interface name="position"/>
+        </joint>
+        <joint name="right_wheel_joint">
+            <command_interface name="velocity">
+                <param name="min">-10</param>
+                <param name="max">10</param>
+            </command_interface>
+            <state_interface name="velocity"/>
+            <state_interface name="position"/>
+        </joint>
+    </ros2_control>
+    <!--
     <ros2_control name="GazeboSystem" type="system">
         <hardware>
@@ -22,4 +52,5 @@
         </joint>
     </ros2_control>
+    -->
     <gazebo>
         <plugin filename="libgazebo_ros2_control.so" name="gazebo_ros2_control">

Commit message: Slam on the robot

File: description/lidar.xacro (robot description, xacro)
@@ -23,4 +23,5 @@
     </link>
     <gazebo reference="laser_frame">
+        <material>Gazebo/Red</material>
         <sensor type="ray" name="laser">
             <pose> 0 0 0 0 0 0 </pose>

File: description/robot_core.xacro (robot description, xacro)
@@ -1,5 +1,5 @@
 <?xml version="1.0"?>
 <robot xmlns:xacro="http://www.ros.org/wiki/xacro">
-<xacro:include filename="inertia_macros.xacro"/>
+    <xacro:include filename="inertia_macros.xacro"/>
     <material name="white">
     <color rgba="1 1 1 1"/>
@@ -19,4 +19,12 @@
     <!-- base link -->
     <link name = "base_link">
+    </link>
+    <!-- BASE_FOOTPRINT LINK -->
+    <joint name="base_footprint_joint" type="fixed">
+        <parent link="base_link"/>
+        <child link="base_footprint"/>
+        <origin xyz="0 0 0" rpy="0 0 0"/>
+    </joint>
+    <link name="base_footprint">
     </link>
     <!-- chasis link -->

File: description/ros2_control.xacro (robot description, xacro)
@@ -15,6 +15,6 @@
         <joint name="left_wheel_joint">
             <command_interface name="velocity">
-                <param name="min">-10</param>
-                <param name="max">10</param>
+                <param name="min">-6</param>
+                <param name="max">6</param>
             </command_interface>
             <state_interface name="velocity"/>
@@ -23,6 +23,6 @@
         <joint name="right_wheel_joint">
             <command_interface name="velocity">
-                <param name="min">-10</param>
-                <param name="max">10</param>
+                <param name="min">-6</param>
+                <param name="max">6</param>
             </command_interface>
             <state_interface name="velocity"/>
